File: KiCAD and GERBER/Pteron56v0.kicad_pcb (KiCad board)
At the start: 2 copper layers, 140.1 x 108.1 mm, 47 parts, among them J1 AudioJack4, J2 AudioJack4, SW10 SW_PUSH, SW12 SW_PUSH, SW13 SW_PUSH, SW14 SW_PUSH, SW15 SW_PUSH, SW17 SW_PUSH, SW18 SW_PUSH, SW19 SW_PUSH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

Commit message: added oled support
Parts:
- added J3: Conn_01x04, usbc_footprint:OLED_4Pin_outline, F.Cu at (103.5, 80.3)
- added JP1: Jumper_NO_Small, SparkFun-Passives:PAD-JUMPER-2-NO_NO_SILK, F.Cu at (102.2, 76.8)
- added JP2: Jumper_NO_Small, SparkFun-Passives:PAD-JUMPER-2-NO_NO_SILK, F.Cu at (100.6, 76.8)
- added JP3: Jumper_NO_Small, SparkFun-Passives:PAD-JUMPER-2-NO_NO_SILK, F.Cu at (98.9, 76.8)
- added JP4: Jumper_NO_Small, SparkFun-Passives:PAD-JUMPER-2-NO_NO_SILK, F.Cu at (97.3, 76.8)
- added JP5: Jumper_NO_Small, SparkFun-Passives:PAD-JUMPER-2-NO_NO_SILK, B.Cu at (102.2, 76.8)
- added JP6: Jumper_NO_Small, SparkFun-Passives:PAD-JUMPER-2-NO_NO_SILK, B.Cu at (100.6, 76.8)
- added JP7: Jumper_NO_Small, SparkFun-Passives:PAD-JUMPER-2-NO_NO_SILK, B.Cu at (98.9, 76.8)
- added JP8: Jumper_NO_Small, SparkFun-Passives:PAD-JUMPER-2-NO_NO_SILK, B.Cu at (97.3, 76.8)
Connections:
- U1 pad 1: (no net) -> /Serial
- U1 pad 5: /Serial -> SDA
- U1 pad 6: (no net) -> SCL
Routing:
- net SDA: track 0.00 -> 35.5 mm, vias 0 -> 1
- net SCL: track 0.00 -> 31.8 mm, vias 0 -> 1
- net /Serial: track 60.6 -> 70.6 mm
- net Net-(J3-Pad4): track 0.00 -> 7.12 mm
- net Net-(J3-Pad1): track 0.00 -> 7.01 mm
- net Net-(J3-Pad3): track 0.00 -> 6.38 mm
- net Net-(J3-Pad2): track 0.00 -> 6.27 mm
- net VCC: track 6.59 -> 12.2 mm, vias 1 -> 3
- net /Row1: track 187.2 -> 192.5 mm
- net /Row2: track 197.0 -> 201.3 mm
- net /Col2: track 181.9 -> 185.7 mm
- net GND: track 6.84 -> 9.07 mm, vias 1 -> 2
- net /Col1: track 200.4 -> 198.6 mm
- net /Row3: track 146.8 -> 147.9 mm
- net /Col4: track 82.8 -> 82.0 mm
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Other:
- board text added: "SDA"

Commit message: added oled, clean silkscreen
Routing:
- net /Col3: track 186.4 -> 185.2 mm

Commit message: add oled, pwm pad, reset switch, moved trrs closer to top, to get simpler casefiles
Parts:
- added PWM_PAD1: Conn_01x03, SparkFun-Connectors:1X03_LONGPADS, B.Cu at (111.8, 55.5)
- added PWM_PAD2: Conn_01x03, SparkFun-Connectors:1X03_LONGPADS, F.Cu at (111.8, 55.5)
- added RST1: SW_PUSH, acheron_Hardware:smdPushBtn, F.Cu at (85.6, 63.6)
- added RST2: SW_PUSH, acheron_Hardware:smdPushBtn, B.Cu at (85.6, 63.6)
- J1, J2: footprint Connector_Audio:Jack_3.5mm_PJ320D_Horizontal -> Keebio-Parts:TRRS-PJ-320A
- moved J1 59.9 mm to (85.5, 44.1)
- moved J2 59.9 mm to (85.5, 44.1), turned to 180 degrees
Connections:
- U1 pad 13: /Col5 -> /PWM
- U1 pad 14: /Col4 -> /Col5
- U1 pad 15: /Col3 -> /Col4
- U1 pad 16: /Col2 -> /Col3
- U1 pad 17: /Col1 -> /Col2
- U1 pad 18: (no net) -> /Col1
- U1 pad 21: (no net) -> VCC
- U1 pad 22: (no net) -> Net-(RST1-Pad1)
- U1 pad 23: (no net) -> GND
- U1 pad 3: (no net) -> GND
- U1 pad 4: (no net) -> GND
Routing:
- net /Serial: track 70.6 -> 9.96 mm, vias 2 -> 0
- net Net-(RST1-Pad1): track 0.00 -> 40.4 mm, vias 0 -> 1
- net /PWM: track 0.00 -> 18.2 mm, vias 0 -> 1
- net GND: track 9.07 -> 22.6 mm, vias 2 -> 3
- net /Row4: track 111.4 -> 108.4 mm
- net /Col1: track 198.6 -> 201.2 mm
- net /Col4: track 82.0 -> 84.5 mm
- net /Col3: track 185.2 -> 187.8 mm
- net /Col2: track 185.7 -> 188.3 mm
- net VCC: track 12.2 -> 13.4 mm
Other:
- outline, holes or cut-outs redrawn
- board text added: "GND"
- board text added: "PWM"
- board text added: "VCC"
