File: KiCAD and GERBER/Pteron36v0.kicad_pcb (KiCad board)
At the start: 2 copper layers, 140.1 x 108.1 mm, 56 parts, among them J1 AudioJack4, J2 AudioJack4, J3 Conn_01x04, SW10 SW_PUSH, SW12 SW_PUSH, SW13 SW_PUSH, SW14 SW_PUSH, SW15 SW_PUSH, SW17 SW_PUSH, SW18 SW_PUSH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

Commit message: updated pcb
Routing:
- net /Col5: track 80.6 -> 96.3 mm
- net /Row3: track 151.3 -> 147.8 mm
- net /Col1: track 201.2 -> 203.4 mm
- net /Col4: track 83.7 -> 85.2 mm
- net /Row2: track 201.5 -> 200.5 mm
