File: KiCAD and GERBER/Pteron36v0.sch (KiCad schematic (older format))
At the start: 62 parts, among them J1 AudioJack4, J2 AudioJack4, J3 Conn_01x04, SW10 SW_PUSH, SW12 SW_PUSH, SW13 SW_PUSH, SW14 SW_PUSH, SW15 SW_PUSH, SW17 SW_PUSH, SW18 SW_PUSH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

Commit message: keebio footprint
Parts:
- SW10, SW12, SW13, SW14, SW15, SW17, SW18, SW19, SW20, SW22, SW23, SW24, SW26, SW27, SW28, SW7, SW8, SW9: footprint User-Submitted:uni-new -> Keebio-Parts:Triple-Dual-1u-LED
Changed lines of the file:
@@
 F 0 "SW7" H 1550 1755 50  0000 C CNN
 F 1 "SW_PUSH" H 1550 1664 50  0000 C CNN
-F 2 "User-Submitted:uni-new" H 1550 1500 60  0001 C CNN
+F 2 "Keebio-Parts:Triple-Dual-1u-LED" H 1550 1500 60  0001 C CNN
 F 3 "" H 1550 1500 60  0000 C CNN
 	1    1550 1500
@@
 F 0 "SW8" H 1550 2405 50  0000 C CNN
 F 1 "SW_PUSH" H 1550 2314 50  0000 C CNN
-F 2 "User-Submitted:uni-new" H 1550 2150 60  0001 C CNN
+F 2 "Keebio-Parts:Triple-Dual-1u-LED" H 1550 2150 60  0001 C CNN
 F 3 "" H 1550 2150 60  0000 C CNN
 	1    1550 2150
@@
 F 0 "SW9" H 1550 3005 50  0000 C CNN
 F 1 "SW_PUSH" H 1550 2914 50  0000 C CNN
-F 2 "User-Submitted:uni-new" H 1550 2750 60  0001 C CNN
+F 2 "Keebio-Parts:Triple-Dual-1u-LED" H 1550 2750 60  0001 C CNN
 F 3 "" H 1550 2750 60  0000 C CNN
 	1    1550 2750
@@
 F 0 "SW12" H 2200 1755 50  0000 C CNN
 F 1 "SW_PUSH" H 2200 1664 50  0000 C CNN
-F 2 "User-Submitted:uni-new" H 2200 1500 60  0001 C CNN
+F 2 "Keebio-Parts:Triple-Dual-1u-LED" H 2200 1500 60  0001 C CNN
 F 3 "" H 2200 1500 60  0000 C CNN
 	1    2200 1500
@@
 F 0 "SW13" H 2200 2405 50  0000 C CNN
 F 1 "SW_PUSH" H 2200 2314 50  0000 C CNN
-F 2 "User-Submitted:uni-new" H 2200 2150 60  0001 C CNN
+F 2 "Keebio-Parts:Triple-Dual-1u-LED" H 2200 2150 60  0001 C CNN
 F 3 "" H 2200 2150 60  0000 C CNN
 	1    2200 2150
@@
 F 0 "SW14" H 2200 3005 50  0000 C CNN
 F 1 "SW_PUSH" H 2200 2914 50  0000 C CNN
-F 2 "User-Submitted:uni-new" H 2200 2750 60  0001 C CNN
+F 2 "Keebio-Parts:Triple-Dual-1u-LED" H 2200 2750 60  0001 C CNN
 F 3 "" H 2200 2750 60  0000 C CNN
 	1    2200 2750
@@
 F 0 "SW17" H 2850 1755 50  0000 C CNN
 F 1 "SW_PUSH" H 2850 1664 50  0000 C CNN
-F 2 "User-Submitted:uni-new" H 2850 1500 60  0001 C CNN
+F 2 "Keebio-Parts:Triple-Dual-1u-LED" H 2850 1500 60  0001 C CNN
 F 3 "" H 2850 1500 60  0000 C CNN
 	1    2850 1500
@@
 F 0 "SW22" H 3500 1755 50  0000 C CNN
 F 1 "SW_PUSH" H 3500 1664 50  0000 C CNN
-F 2 "User-Submitted:uni-new" H 3500 1500 60  0001 C CNN
+F 2 "Keebio-Parts:Triple-Dual-1u-LED" H 3500 1500 60  0001 C CNN
 F 3 "" H 3500 1500 60  0000 C CNN
 	1    3500 1500
@@
 F 0 "SW18" H 2850 2405 50  0000 C CNN
 F 1 "SW_PUSH" H 2850 2314 50  0000 C CNN
-F 2 "User-Submitted:uni-new" H 2850 2150 60  0001 C CNN
+F 2 "Keebio-Parts:Triple-Dual-1u-LED" H 2850 2150 60  0001 C CNN
 F 3 "" H 2850 2150 60  0000 C CNN
 	1    2850 2150
@@
 F 0 "SW19" H 2850 3005 50  0000 C CNN
 F 1 "SW_PUSH" H 2850 2914 50  0000 C CNN
-F 2 "User-Submitted:uni-new" H 2850 2750 60  0001 C CNN
+F 2 "Keebio-Parts:Triple-Dual-1u-LED" H 2850 2750 60  0001 C CNN
 F 3 "" H 2850 2750 60  0000 C CNN
 	1    2850 2750
@@
 F 0 "SW23" H 3500 2405 50  0000 C CNN
 F 1 "SW_PUSH" H 3500 2314 50  0000 C CNN
-F 2 "User-Submitted:uni-new" H 3500 2150 60  0001 C CNN
+F 2 "Keebio-Parts:Triple-Dual-1u-LED" H 3500 2150 60  0001 C CNN
 F 3 "" H 3500 2150 60  0000 C CNN
 	1    3500 2150
@@
 F 0 "SW24" H 3500 3005 50  0000 C CNN
 F 1 "SW_PUSH" H 3500 2914 50  0000 C CNN
-F 2 "User-Submitted:uni-new" H 3500 2750 60  0001 C CNN
+F 2 "Keebio-Parts:Triple-Dual-1u-LED" H 3500 2750 60  0001 C CNN
 F 3 "" H 3500 2750 60  0000 C CNN
 	1    3500 2750
@@
 F 0 "SW26" H 4150 1755 50  0000 C CNN
 F 1 "SW_PUSH" H 4150 1664 50  0000 C CNN
-F 2 "User-Submitted:uni-new" H 4150 1500 60  0001 C CNN
+F 2 "Keebio-Parts:Triple-Dual-1u-LED" H 4150 1500 60  0001 C CNN
 F 3 "" H 4150 1500 60  0000 C CNN
 	1    4150 1500
@@
 F 0 "SW27" H 4150 2405 50  0000 C CNN
 F 1 "SW_PUSH" H 4150 2314 50  0000 C CNN
-F 2 "User-Submitted:uni-new" H 4150 2150 60  0001 C CNN
+F 2 "Keebio-Parts:Triple-Dual-1u-LED" H 4150 2150 60  0001 C CNN
 F 3 "" H 4150 2150 60  0000 C CNN
 	1    4150 2150
@@
 F 0 "SW28" H 4150 3005 50  0000 C CNN
 F 1 "SW_PUSH" H 4150 2914 50  0000 C CNN
-F 2 "User-Submitted:uni-new" H 4150 2750 60  0001 C CNN
+F 2 "Keebio-Parts:Triple-Dual-1u-LED" H 4150 2750 60  0001 C CNN
 F 3 "" H 4150 2750 60  0000 C CNN
 	1    4150 2750
@@
 F 0 "SW10" H 1550 3605 50  0000 C CNN
 F 1 "SW_PUSH" H 1550 3514 50  0000 C CNN
-F 2 "User-Submitted:uni-new" H 1550 3350 60  0001 C CNN
+F 2 "Keebio-Parts:Triple-Dual-1u-LED" H 1550 3350 60  0001 C CNN
 F 3 "" H 1550 3350 60  0000 C CNN
 	1    1550 3350
@@
 F 0 "SW15" H 2200 3605 50  0000 C CNN
 F 1 "SW_PUSH" H 2200 3514 50  0000 C CNN
-F 2 "User-Submitted:uni-new" H 2200 3350 60  0001 C CNN
+F 2 "Keebio-Parts:Triple-Dual-1u-LED" H 2200 3350 60  0001 C CNN
 F 3 "" H 2200 3350 60  0000 C CNN
 	1    2200 3350
@@
 F 0 "SW20" H 2850 3605 50  0000 C CNN
 F 1 "SW_PUSH" H 2850 3514 50  0000 C CNN
-F 2 "User-Submitted:uni-new" H 2850 3350 60  0001 C CNN
+F 2 "Keebio-Parts:Triple-Dual-1u-LED" H 2850 3350 60  0001 C CNN
 F 3 "" H 2850 3350 60  0000 C CNN
 	1    2850 3350
