File: lowprofile-pcb/Pteron36v0.kicad_pcb (KiCad board)
At the start: 2 copper layers, 123.5 x 95.6 mm, 46 parts, among them J1 AudioJack4, J2 AudioJack4, SW10 SW_PUSH, SW12 SW_PUSH, SW13 SW_PUSH, SW14 SW_PUSH, SW15 SW_PUSH, SW17 SW_PUSH, SW18 SW_PUSH, SW19 SW_PUSH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

Commit message: introduce the snapable pcb with 4 config of keyboard possible
Parts:
- removed LOGO1, LOGO2: LOGO-OTL, personal-logo:miryoku-kicad-small
- removed RST1, RST2: SW_PUSH, acheron_Hardware:smdPushBtn
- added JP1: JUMPER-PAD-2-NO, Jumper:SolderJumper-2_P1.3mm_Open_Pad1.0x1.5mm, F.Cu at (125.6, 66.2)
- added JP2: JUMPER-PAD-2-NO, Jumper:SolderJumper-2_P1.3mm_Open_Pad1.0x1.5mm, B.Cu at (125.6, 66.2)
- moved LOGO3 22.3 mm to (125.9, 91.2), turned to 37 degrees
- moved LOGO4 20.7 mm to (125.1, 89.9), turned to -10 degrees
Routing:
- net Net-(U1-Pad22): track 48.3 -> 30.9 mm
- net GND: track 11.3 -> 5.06 mm
