File: lowprofile-pcb/Pteron36v0.kicad_sch (KiCad schematic)
At the start: 46 parts, among them J1 AudioJack4, J2 AudioJack4, SW10 SW_PUSH, SW12 SW_PUSH, SW13 SW_PUSH, SW14 SW_PUSH, SW15 SW_PUSH, SW17 SW_PUSH, SW18 SW_PUSH, SW19 SW_PUSH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

Commit message: add stl for 38 key variant case, add 1.5 u on lowprofile keyboard
Parts:
- removed LOGO1, LOGO2: LOGO-OTL, personal-logo:miryoku-kicad-small, symbol SparkFun-Aesthetics:LOGO-OTL
- added SW1: SW_PUSH, keyswitches:PG1350_reversible, symbol keyboard_parts:SW_PUSH
Connections:
- net Row4: now also SW1.1
- net at D20.2 (A), SW20.2: now also SW1.2
Changed lines of the file:
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@@
   (junction (at 64.77 62.23) (diameter 1.016) (color 0 0 0 0))
   (junction (at 64.77 77.47) (diameter 1.016) (color 0 0 0 0))
+  (junction (at 64.77 85.09) (diameter 1.016) (color 0 0 0 0))
   (junction (at 68.58 60.96) (diameter 1.016) (color 0 0 0 0))
   (junction (at 68.58 76.2) (diameter 1.016) (color 0 0 0 0))
   (junction (at 68.58 91.44) (diameter 1.016) (color 0 0 0 0))
+  (junction (at 80.01 89.535) (diameter 1.016) (color 0 0 0 0))
   (junction (at 81.28 30.48) (diameter 1.016) (color 0 0 0 0))
   (junction (at 81.28 46.99) (diameter 1.016) (color 0 0 0 0))
@@
     (stroke (width 0) (type solid) (color 0 0 0 0))
   )
+  (wire (pts (xy 64.77 85.09) (xy 64.77 89.535))
+    (stroke (width 0) (type solid) (color 0 0 0 0))
+  )
   (wire (pts (xy 68.58 44.45) (xy 68.58 60.96))
     (stroke (width 0) (type solid) (color 0 0 0 0))
@@
     (stroke (width 0) (type solid) (color 0 0 0 0))
   )
-  (wire (pts (xy 80.01 85.09) (xy 80.01 91.44))
+  (wire (pts (xy 80.01 85.09) (xy 80.01 89.535))
+    (stroke (width 0) (type solid) (color 0 0 0 0))
+  )
+  (wire (pts (xy 80.01 89.535) (xy 80.01 91.44))
     (stroke (width 0) (type solid) (color 0 0 0 0))
   )
@@
     (pin "2")
   )
+  (symbol (lib_id "keyboard_parts:SW_PUSH") (at 72.39 89.535 0) (unit 1)
+    (in_bom yes) (on_board yes)
+    (property "Reference" "SW1" (id 0) (at 72.39 83.058 0))
+    (property "Value" "SW_PUSH" (id 1) (at 72.39 85.3694 0))
+    (property "Footprint" "keyswitches:PG1350_reversible" (id 2) (at 72.39 89.535 0)
+      (effects (font (size 1.524 1.524)) hide)
+    )
+    (property "Datasheet" "" (id 3) (at 72.39 89.535 0)
+      (effects (font (size 1.524 1.524)))
+    )
+    (pin "1")
+    (pin "2")
+  )
   (symbol (lib_id "keyboard_parts:SW_PUSH") (at 88.9 38.1 0) (unit 1)
     (in_bom yes) (on_board yes)
@@
     (pin "1")
     (pin "2")
-  )
-  (symbol (lib_id "SparkFun-Aesthetics:LOGO-OTL") (at 234.95 76.2 0) (unit 1)
-    (in_bom yes) (on_board yes)
-    (property "Reference" "LOGO1" (id 0) (at 234.95 76.2 0)
-      (effects (font (size 1.27 1.27)) hide)
-    )
-    (property "Value" "LOGO-OTL" (id 1) (at 234.95 76.2 0)
-      (effects (font (size 1.27 1.27)) hide)
-    )
-    (property "Footprint" "personal-logo:miryoku-kicad-small" (id 2) (at 235.712 72.39 0)
-      (effects (font (size 0.508 0.508)) hide)
-    )
-    (property "Datasheet" "" (id 3) (at 234.95 76.2 0)
-      (effects (font (size 1.27 1.27)) hide)
-    )
-  )
-  (symbol (lib_id "SparkFun-Aesthetics:LOGO-OTL") (at 234.95 86.36 0) (unit 1)
-    (in_bom yes) (on_board yes)
-    (property "Reference" "LOGO2" (id 0) (at 234.95 86.36 0)
-      (effects (font (size 1.27 1.27)) hide)
-    )
-    (property "Value" "LOGO-OTL" (id 1) (at 234.95 86.36 0)
-      (effects (font (size 1.27 1.27)) hide)
-    )
-    (property "Footprint" "personal-logo:miryoku-kicad-small" (id 2) (at 235.712 82.55 0)
-      (effects (font (size 0.508 0.508)) hide)
-    )
-    (property "Datasheet" "" (id 3) (at 234.95 86.36 0)
-      (effects (font (size 1.27 1.27)) hide)
-    )
   )
   (symbol (lib_id "SparkFun-Aesthetics:LOGO-OTL") (at 251.46 76.2 0) (unit 1)
@@
       (reference "J2") (unit 1) (value "AudioJack4") (footprint "Keebio-Parts:TRRS-PJ-320A")
     )
-    (path "/00000000-0000-0000-0000-0000607a2bee"
-      (reference "LOGO1") (unit 1) (value "LOGO-OTL") (footprint "personal-logo:miryoku-kicad-small")
-    )
-    (path "/00000000-0000-0000-0000-0000607a2653"
-      (reference "LOGO2") (unit 1) (value "LOGO-OTL") (footprint "personal-logo:miryoku-kicad-small")
-    )
     (path "/e4d4d865-3cb1-431d-b18c-3cc2928a93c9"
       (reference "LOGO3") (unit 1) (value "LOGO-OTL") (footprint "personal-logo:peacock-medium")
@@
       (reference "RST2") (unit 1) (value "SW_PUSH") (footprint "acheron_Hardware:smdPushBtn")
     )
+    (path "/402851d8-0ae4-4da3-93c1-370c6cc5e9c2"
+      (reference "SW1") (unit 1) (value "SW_PUSH") (footprint "keyswitches:PG1350_reversible")
+    )
     (path "/00000000-0000-0000-0000-000060963566"
