File: universal-pcb/Pteron36v0.kicad_pcb (KiCad board)
At the start: 2 copper layers, 140.1 x 108.1 mm, 62 parts, among them J1 AudioJack4, J2 AudioJack4, J3 Conn_01x04, SW10 SW_PUSH, SW12 SW_PUSH, SW13 SW_PUSH, SW14 SW_PUSH, SW15 SW_PUSH, SW17 SW_PUSH, SW18 SW_PUSH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

Commit message: ready for multi slot version of pcb
Parts:
- removed H3, H6: MountingHole, MountingHole:MountingHole_2.2mm_M2
- added D25: 1N4148, Keebio-Parts:Diode-dual, F.Cu at (37.8, 91.8)
- added SW25: SW_PUSH, Keebio-Parts:Triple-Dual-1u-LED, F.Cu at (143.8, 114.3)
Routing:
- net /Col1: track 222.2 -> 152.4 mm
- net /Row4: track 309.4 -> 251.1 mm
- net /Col2: track 220.2 -> 169.1 mm
- net /Col3: track 196.5 -> 162.5 mm
- net Net-(SW25-Pad2): track 0.00 -> 11.3 mm
Other:
- outline, holes or cut-outs redrawn
- net class Default removed

Commit message: eureka of super finish
Parts:
- removed H1: MountingHole, MountingHole:MountingHole_2.2mm_M2
- moved D25 143.4 mm to (175.1, 133.4)
- moved D20 44.6 mm to (122.8, 151.4), turned to 37.5 degrees
- moved PWM_PAD1 33.8 mm to (142.9, 71.6)
- moved PWM_PAD2 33.8 mm to (142.9, 71.6)
- moved D7 33.8 mm to (219.3, 77.6)
- moved H2 33.8 mm to (209.7, 74.7)
- moved SW13 33.8 mm to (209.7, 84.3)
- moved JP1 33.8 mm to (134.5, 93.0)
- moved JP5 33.8 mm to (134.5, 93.0)
- moved D18 33.8 mm to (181.1, 85.0)
- moved SW26 33.8 mm to (152.5, 69.1)
- moved SW27 33.8 mm to (152.5, 88.1)
- moved D22 33.8 mm to (162.1, 71.6)
- moved SW8 33.8 mm to (228.7, 93.9)
- moved D12 33.8 mm to (200.2, 69.0)
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Routing:
- net /Row4: track 251.1 -> 335.0 mm
- net /Col1: track 152.4 -> 214.8 mm
- net /Col2: track 169.1 -> 218.5 mm
- net /Col4: track 76.2 -> 121.8 mm, vias 1 -> 3
- net /Col3: track 162.5 -> 189.2 mm, vias 0 -> 1
- net /Row1: track 202.0 -> 177.1 mm
- net Net-(SW25-Pad2): track 11.3 -> 23.7 mm
- net Net-(D24-Pad2): track 34.9 -> 28.0 mm
- net Net-(D20-Pad2): track 24.2 -> 28.5 mm
- net /Row2: track 333.9 -> 333.0 mm
- net Net-(D17-Pad2): track 39.3 -> 38.4 mm
- net Net-(D15-Pad2): track 26.2 -> 26.8 mm
Other:
- board size 140.1 x 108.1 mm -> 135.4 x 104.4 mm
- board text removed: "Based on Pteron keyboard by Fsund Based on Pteron pcb by Kraken-Jokes"
